File: ch348q/ch348q.kicad_sch (KiCad schematic)
At the start: 16 parts, among them J1 Conn_01x10_Pin, J2 Conn_02x03_Counter_Clockwise, SW1 SW_Push, U2 CH348L, Y1 Crystal

Commit message: feat: update.
Parts:
- added C11, C12, C14, C15: 1uF, Capacitor_SMD:C_0402_1005Metric, symbol Device:C
- added C13: 100nF, Capacitor_SMD:C_0402_1005Metric, symbol Device:C
- added C16: 10nF, Capacitor_SMD:C_0402_1005Metric, symbol Device:C
- added D1: LED_GREEN, LED_SMD:LED_Cree-PLCC4_2x2mm_CW, symbol Device:LED
- added D2: LED_BLUE, LED_SMD:LED_Cree-PLCC4_2x2mm_CW, symbol Device:LED
- added D3: LED_YELLOW, LED_SMD:LED_Cree-PLCC4_2x2mm_CW, symbol Device:LED
- added D4: LED_RED, LED_SMD:LED_Cree-PLCC4_2x2mm_CW, symbol Device:LED
- added F1: 500mA, Fuse:Fuse_0805_2012Metric, symbol Device:Fuse
- added IC1: SGM2019-3.3YN5G_TR, Package_TO_SOT_SMD:SOT-23-5, symbol power_ic:SGM2019-3.3YN5G_TR
- added J10: USB_C_Receptacle_USB2.0_16P, Connector_USB:USB_C_Receptacle_GCT_USB4105-xx-A_16P_TopMnt_Horizontal, symbol Connector:USB_C_Receptacle_USB2.0_16P
- added J3, J4, J5, J6, J7, J8, J9: Conn_01x10_Pin, Connector_PinHeader_2.54mm:PinHeader_1x10_P2.54mm_Vertical_SMD_Pin1Left, symbol Connector:Conn_01x10_Pin
- added R2: 22K7, Resistor_SMD:R_0402_1005Metric, symbol Device:R
- added R3: 33K5, Resistor_SMD:R_0402_1005Metric, symbol Device:R
- added R4: 50K, Resistor_SMD:R_0402_1005Metric, symbol Device:R
- added R5: 10K, Resistor_SMD:R_0402_1005Metric, symbol Device:R
- added R6, R7: 5K1, Resistor_SMD:R_0402_1005Metric, symbol Device:R
- added R8, R9: 4K7, Resistor_SMD:R_0402_1005Metric, symbol Device:R
- added SW2: SW_Nidec_CAS-120A1, Button_Switch_SMD:Nidec_Copal_CAS-120A, symbol Switch:SW_Nidec_CAS-120A1
- added U1: ~, Package_DFN_QFN:TDFN-6-1EP_2.5x2.5mm_P0.65mm_EP1.3x2mm, symbol power_ic:SGM2060-ADJ
- R1: value 4k7 -> 4K7
- renumbered J2 to J1, J1 to J2
Connections:
- net +3V3: now also C15.1, IC1.5 (OUT), SW2.3 (A)
- net ACT: now also D1.1 (K)
- net CFG: now also SW2.2 (B)
- net CTS0/GPIO0: now also J2.6 (Pin_6)
- net CTS1/GPIO2: now also J3.6 (Pin_6)
- net DCD0/GPIO26: now also J2.10 (Pin_10)
- net DCD1/GPIO28: now also J3.10 (Pin_10)
- net DSR0/GPIO24: now also J2.8 (Pin_8)
- net DSR1/GPIO27: now also J3.8 (Pin_8)
- net DTR0/TNOW0/GPIO8: now also J2.7 (Pin_7)
- net DTR1/TNOW1/GPIO9: now also J3.7 (Pin_7)
- net GND: now also J2.2 (Pin_2), U2.37 (GND), C11.2, C12.2, C14.2, C15.2, C16.1, D4.1 (K), IC1.2 (GND), J10.A1 (GND), J10.A12 (GND), J10.B1 (GND), J10.B12 (GND), J10.S1 (SHIELD), J3.2 (Pin_2), J4.2 (Pin_2), J5.2 (Pin_2), J6.2 (Pin_2), J7.2 (Pin_2), J8.2 (Pin_2), J9.2 (Pin_2), R5.2, R6.2, R7.2, R8.1, R9.2, U1.3 (GND), U1.7 (PAD)
- net RI0/GPIO25: now also J2.9 (Pin_9)
- net RI1/GPIO29: now also J3.9 (Pin_9)
- net RTS0/GPIO1: now also J2.5 (Pin_5)
- net RTS1/GPIO3: now also J3.5 (Pin_5)
- net RXD0: now also J2.3 (Pin_3)
- net RXD1: now also J3.3 (Pin_3)
- net RXD2: now also J4.3 (Pin_3)
- net RXD3: now also J5.3 (Pin_3)
- net RXD4: now also J6.3 (Pin_3)
- net RXD5: now also J7.3 (Pin_3)
- net RXD6: now also J8.3 (Pin_3)
- net RXD7: now also J9.3 (Pin_3)
- net RX_S: now also D3.1 (K)
- net TXD0: now also J2.4 (Pin_4)
- net TXD1: now also J3.4 (Pin_4)
- net TXD2: now also J4.4 (Pin_4)
- net TXD3: now also J5.4 (Pin_4)
- net TXD4: now also J6.4 (Pin_4)
- net TXD5: now also J7.4 (Pin_4)
- net TXD6: now also J8.4 (Pin_4)
- net TXD7: now also J9.4 (Pin_4)
- net TX_S: now also D2.1 (K)
- net UD+: now also J10.A6 (D+), J10.B6 (D+)
- net UD-: now also J10.A7 (D-), J10.B7 (D-)
- net VIO: now also J2.1 (Pin_1), C12.1, C13.1, D1.2 (A), D2.2 (A), D3.2 (A), D4.2 (A), J3.1 (Pin_1), J4.1 (Pin_1), J5.1 (Pin_1), J6.1 (Pin_1), J7.1 (Pin_1), J8.1 (Pin_1), J9.1 (Pin_1), U1.1 (OUT)
- net at J1.4 (Pin_4): now also R4.1
- net at J1.5 (Pin_5): now also R3.1
- net at J1.6 (Pin_6): now also R2.1
- net TEST: no longer names the net of U2.94 (TEST)
- net TEST: now also R8.2
- new net: J10.A5 (CC1), R6.1
- new net: J10.B5 (CC2), R7.1
- new net: C16.2, IC1.4 (BP/FB)
- new net: R9.1, SW2.1 (C)
- new net +5V: C11.1, C14.1, F1.2, IC1.1 (IN), IC1.3 (EN), U1.4 (EN), U1.6 (IN)
- new net CTS2/GPIO4: J4.6 (Pin_6)
- new net CTS3/GPIO6: J5.6 (Pin_6)
- new net CTS4/GPIO12: J6.6 (Pin_6)
- new net CTS5/GPIO14: J7.6 (Pin_6)
- new net CTS6/GPIO16: J8.6 (Pin_6)
- new net CTS7/GPIO18: J9.6 (Pin_6)
- new net DCD2/GPIO31: J4.10 (Pin_10)
- new net DCD3/GPIO34: J5.10 (Pin_10)
- new net DCD4/GPIO37: J6.10 (Pin_10)
- new net DCD5/GPIO40: J7.10 (Pin_10)
- new net DCD6/GPIO43: J8.10 (Pin_10)
- new net DCD7/GPIO46: J9.10 (Pin_10)
- new net DSR2/GPIO30: J4.8 (Pin_8)
- new net DSR3/GPIO33: J5.8 (Pin_8)
- new net DSR4/GPIO36: J6.8 (Pin_8)
- new net DSR5/GPIO39: J7.8 (Pin_8)
- new net DSR6/GPIO42: J8.8 (Pin_8)
- new net DSR7/GPIO45: J9.8 (Pin_8)
- new net DTR2/TNOW2/GPIO10: J4.7 (Pin_7)
- new net DTR3/TNOW3/GPIO11: J5.7 (Pin_7)
- new net DTR4/TNOW4/GPIO20: J6.7 (Pin_7)
- new net DTR5/TNOW5/GPIO21: J7.7 (Pin_7)
- new net DTR6/TNOW6/GPIO22: J8.7 (Pin_7)
- new net DTR7/TNOW7/GPIO23: J9.7 (Pin_7)
- new net RI2/GPIO32: J4.9 (Pin_9)
- new net RI3/GPIO35: J5.9 (Pin_9)
- new net RI4/GPIO38: J6.9 (Pin_9)
- new net RI5/GPIO41: J7.9 (Pin_9)
- new net RI6/GPIO44: J8.9 (Pin_9)
- new net RI7/GPIO47: J9.9 (Pin_9)
- new net RTS2/GPIO5: J4.5 (Pin_5)
- new net RTS3/GPIO7: J5.5 (Pin_5)
- new net RTS4/GPIO13: J6.5 (Pin_5)
- new net RTS5/GPIO15: J7.5 (Pin_5)
- new net RTS6/GPIO17: J8.5 (Pin_5)
- new net RTS7/GPIO19: J9.5 (Pin_5)
- new net VBUS: F1.1, J10.A4 (VBUS), J10.A9 (VBUS), J10.B4 (VBUS), J10.B9 (VBUS)
- new net VFB: C13.2, R2.2, R3.2, R4.2, R5.1, U1.2 (FB)
- no-connect marks 11 -> 13
Other:
- note added: "20251004"
- note added: "V1.0"
- note added: "V_{OUT}=V_{ADJ}×(1+R2/R3) V_{ADJ}=0.55V R2=22.7kΩ,1.8V R3=35.5kΩ,2.5V R4=50kΩ,3.3V"
- note added: "ch348q_usb_to_8_uart"
- moved on the sheet: J1, J2
